Commit message: woc调这个还挺累的

File: src/mujuco_rotating/engineer_module/meshes/arm/engineer_v2.urdf (robot description, URDF)
Before this commit: robot engineer, 18 links, 17 joints
Links:
- removed link Link7_rot_y
- removed link Link7_rot_z
- removed link Link7_trans_x
- removed link Link7_trans_y
- removed link Link7_trans_z
Joints:
- removed joint rot_x
- removed joint rot_y
- removed joint rot_z
- removed joint trans_x
- removed joint trans_y
- removed joint trans_z
- added joint J_box: type fixed, parent Link7, child LinkB, origin xyz=0 0 0  rpy=0 0 0
- joint Joint5: origin xyz=0 0 0 rpy=-1.5708 0 -3.1416 -> xyz=0 0 0 rpy=-1.5708 1.5708 -3.1416; type revolute -> fixed
